File: revlp/one42/one42_pcb/one42.kicad_pcb (KiCad board)
At the start: 2 copper layers, 265.7 x 104.1 mm, 117 parts, among them J1 Conn_01x04_Female, Q1 AO3401A, SW1 SW_SPST, SW10 SW_Push, SW11 SW_Push, SW12 SW_Push, SW13 SW_Push, SW14 SW_Push, SW15 SW_Push, SW16 SW_Push, SW17 SW_Push, SW18 SW_Push, SW19 SW_Push, SW2 SW_Push, SW20 SW_Push, SW21 SW_Push, SW22 SW_Push, SW23 SW_Push, SW24 SW_Push, SW25 SW_Push, SW26 SW_Push, SW27 SW_Push, SW28 SW_Push, SW29 SW_Push, SW3 SW_Push, SW30 SW_Push, SW31 SW_Push, SW32 SW_Push, SW33 SW_Push, SW34 SW_Push, SW35 SW_Push, SW36 SW_Push, SW37 SW_Push, SW38 SW_SPDT, SW4 SW_Push, SW5 SW_Push, SW6 SW_Push, SW7 SW_Push, SW8 SW_Push, SW9 SW_Push, U2 AP2112K-3.3, U3 TP4054, U4 nRF52840_holyiot_18010

Commit message: [keyboard] One42: Long Live Ahokore!
Parts:
- removed BT2: Battery_Cell, custom-parts:custombatteryconnector
- removed G***: LOGO, custom-parts:fantail-on
- removed G***: LOGO, custom-parts:fantail-off
- removed G***: LOGO, custom-parts:fantail-v22
- removed G***: LOGO, custom-parts:fantail-dezli2
- removed G***: LOGO, custom-parts:fantail-fantail1
- removed G***: LOGO, custom-parts:fantail-ahokore5
- removed G***: LOGO, custom-parts:ahokore
- removed H10, H9: MountingHole_Pad, MountingHole:MountingHole_2.2mm_M2_DIN965_Pad
- removed SW1: SW_SPST, custom-parts:custom-reset-switch
- removed SW10, SW11, SW12, SW13, SW14, SW15, SW16, SW17, SW18, SW19, SW2, SW20, SW21, SW22, SW23, SW24, SW25, SW26, SW27, SW28, SW29, SW3, SW30, SW31, SW32, SW33, SW34, SW35, SW36, SW37, SW4, SW5, SW6, SW7, SW8, SW9: SW_Push, switches:Choc_PG1350_Choc_Spacing
- removed SW38: SW_SPDT, custom-parts:OS102011MA1QN1
- added D41: D_Small, Diode_SMD:D_SOD-123, F.Cu at (65.7, 114.4)
- added D42: D_Small, Diode_SMD:D_SOD-123, F.Cu at (80.2, 102.5)
- added D43: SR05, Package_TO_SOT_SMD:SOT-143, F.Cu at (37.7, 55.2)
- added D44: 1N5819, Diode_SMD:D_SOD-123, F.Cu at (37.0, 77.4)
- added D45: powerLED, Diode_SMD:D_0805_2012Metric, F.Cu at (44.7, 46.0)
- added D46: statusLED, Diode_SMD:D_0805_2012Metric, F.Cu at (30.7, 46.0)
- added JP1: EncoderPolarity, Jumper:SolderJumper-3_P1.3mm_Open_RoundedPad1.0x1.5mm, F.Cu at (18.0, 114.6)
- added JP3: Reset, Jumper:SolderJumper-2_P1.3mm_Open_RoundedPad1.0x1.5mm, F.Cu at (51.1, 51.6)
- added SW44: SW_SPDT, keebLib:switch_SSSS811101, F.Cu at (63.7, 43.2)
- added SwA00: SW_Push, keebLib:pg1353, F.Cu at (-67.4, 44.7)
- added SwA01: SW_Push, keebLib:pg1353, F.Cu at (-49.2, 49.5)
- added SwA02: SW_Push, keebLib:pg1353, F.Cu at (-28.5, 44.7)
- added SwA03: SW_Push, keebLib:pg1353, F.Cu at (-9.01, 44.7)
- added SwA04: SW_Push, keebLib:pg1353, F.Cu at (7.84, 54.4)
- added SwA05: SW_Push, keebLib:pg1353, F.Cu at (24.7, 64.1)
- added SwA06: SW_Push, keebLib:pg1353, F.Cu at (50.7, 64.1)
- added SwA07: SW_Push, keebLib:pg1353, F.Cu at (67.6, 54.4)
- added SwA08: SW_Push, keebLib:pg1353, F.Cu at (84.4, 44.7)
- added SwA09: SW_Push, keebLib:pg1353, F.Cu at (103.9, 44.6)
- added SwA10: SW_Push, keebLib:pg1353, F.Cu at (124.7, 49.5)
- added SwA11: SW_Push, keebLib:pg1353, F.Cu at (142.8, 44.7)
- added SwB00: SW_Push, keebLib:pg1353, F.Cu at (-72.3, 62.8)
- added SwB01: SW_Push, keebLib:pg1353, F.Cu at (-54.1, 67.7)
- added SwB02: SW_Push, keebLib:pg1353, F.Cu at (-33.3, 62.8)
- added SwB03: SW_Push, keebLib:pg1353, F.Cu at (-13.9, 62.8)
- added SwB04: SW_Push, keebLib:pg1353, F.Cu at (2.98, 72.6)
- added SwB05: SW_Push, keebLib:pg1353, F.Cu at (19.8, 82.3)
- added SwB06: SW_Push, keebLib:pg1353, F.Cu at (55.6, 82.3)
- added SwB07: SW_Push, keebLib:pg1353, F.Cu at (72.4, 72.6)
- added SwB08: SW_Push, keebLib:pg1353, F.Cu at (89.3, 62.8)
- added SwB09: SW_Push, keebLib:pg1353, F.Cu at (108.8, 62.8)
- added SwB10: SW_Push, keebLib:pg1353, F.Cu at (129.5, 67.7)
- added SwB11: SW_Push, keebLib:pg1353, F.Cu at (147.7, 62.8)
- added SwC00: SW_Push, keebLib:pg1353, F.Cu at (-77.1, 81.0)
- added SwC01: SW_Push, keebLib:pg1353, F.Cu at (-59.0, 85.9)
- added SwC02: SW_Push, keebLib:pg1353, F.Cu at (-38.2, 81.0)
- added SwC03: SW_Push, keebLib:pg1353, F.Cu at (-18.7, 81.0)
- added SwC04: SW_Push, keebLib:pg1353, F.Cu at (-1.89, 90.7)
- added SwC05: SW_Push, keebLib:pg1353, F.Cu at (15.0, 100.5)
- added SwC06: SW_Push, keebLib:pg1353, F.Cu at (60.5, 100.5)
- added SwC07: SW_Push, keebLib:pg1353, F.Cu at (77.3, 90.7)
- added SwC08: SW_Push, keebLib:pg1353, F.Cu at (94.2, 81.0)
- added SwC09: SW_Push, keebLib:pg1353, F.Cu at (113.6, 81.0)
- added SwC10: SW_Push, keebLib:pg1353, F.Cu at (134.4, 85.8)
- added SwC11: SW_Push, keebLib:pg1353, F.Cu at (152.6, 81.0)
- added SwD03: Rotary_Encoder_Switch, keebLib:pg1353_ec11rotSw, F.Cu at (-11.0, 110.6)
- added SwD04: SW_Push, keebLib:pg1353, F.Cu at (8.39, 119.2)
- added SwD05: SW_Push, keebLib:pg1353, F.Cu at (24.9, 132.5)
- added SwD06: SW_Push, keebLib:pg1353, F.Cu at (50.6, 132.5)
- added SwD07: SW_Push, keebLib:pg1353, F.Cu at (67.0, 119.2)
- added SwD08: Rotary_Encoder_Switch, keebLib:pg1353_ec11rotSw, F.Cu at (86.4, 110.6)
- added U1: TP4054, Package_TO_SOT_SMD:SOT-23-5, F.Cu at (59.4, 110.2)
- BT1: footprint custom-parts:JST_PH_S2B-PH-K_1x02_P2.00mm_Horizontal -> keebLib:cell_pads
- C2: value 4.7n -> 1uF; footprint Capacitor_SMD:C_1206_3216Metric -> Capacitor_SMD:C_0805_2012Metric
- C4: value 1uF -> 4.7n; footprint Capacitor_SMD:C_0805_2012Metric -> Capacitor_SMD:C_1206_3216Metric
- D1: value 1N5819 -> D_Small
- D2: value POWERLED -> D_Small; footprint Diode_SMD:D_0805_2012Metric -> Diode_SMD:D_SOD-123
- D39: value LED_Small -> D_Small; footprint Diode_SMD:D_0805_2012Metric -> Diode_SMD:D_SOD-123
- D40: value SR05 -> D_Small; footprint Package_TO_SOT_SMD:SOT-143 -> Diode_SMD:D_SOD-123
- H1, H2, H3, H4, H5, H6, H7, H8: value MountingHole_Pad -> MountingHole; footprint MountingHole:MountingHole_2.2mm_M2_DIN965_Pad -> MountingHole:MountingHole_2.2mm_M2_Pad
- R3: value 10k -> 5.1k
- R4: value 1k -> 10k
- R5: value 5.1k -> 1k
- R7: value 806k -> 1k
- R8: value 2M -> 806k
- R9: value 1k -> 2M
- U3: value TP4054 -> nRF52840_holyiot_18010; footprint Package_TO_SOT_SMD:SOT-23-5 -> keebMCU:nRF52840_holyiot_18010_HS_simple
- U4: value nRF52840_holyiot_18010 -> One42; footprint kicad-keyboard-parts:nRF52840_holyiot_18010 -> one42:one42
- USB1: footprint Type-C:HRO-TYPE-C-31-M-12-HandSoldering -> keebMCU:USB_C_Receptacle_HRO_TYPE-C-31-M-12_handsolder
- moved D1 218.3 mm to (-66.1, 39.9), turned to 165 degrees
- moved H5 218.2 mm to (37.7, 125.6)
- moved H7 210.3 mm to (37.7, 63.5)
- moved D30 199.2 mm to (16.3, 95.7), turned to 165 degrees
- moved D37 199.0 mm to (-17.3, 102.3), turned to 180 degrees
- moved D29 194.8 mm to (-0.60, 85.9), turned to 165 degrees
- moved D38 194.5 mm to (10.0, 113.5), turned to 165 degrees
- moved D2 192.5 mm to (-48.0, 44.7), turned to 165 degrees
- moved D28 191.9 mm to (-17.5, 76.2), turned to 165 degrees
- moved D31 174.6 mm to (59.1, 95.6), turned to -165 degrees
- moved D32 172.1 mm to (76.0, 85.9), turned to -165 degrees
- moved H8 165.4 mm to (1.27, 104.2)
- moved D18 155.9 mm to (21.1, 77.5), turned to 165 degrees
- moved D39 154.9 mm to (27.5, 127.2), turned to 150 degrees
- moved D19 142.3 mm to (54.3, 77.5), turned to -165 degrees
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Connections:
- BT1 pad 1: Net-(BT1-Pad1) -> VBAT
- BT1 pad 2: GND -> Net-(BT1-Pad2)
- C1 pad 1: VBAT -> GND
- C1 pad 2: GND -> VBAT
- C2 pad 1: GND -> VDD_NRF
- C2 pad 2: Earth -> GND
- C3 pad 1: VDD_NRF -> /PVIN
- C4 pad 1: Net-(C4-Pad1) -> GND
- C4 pad 2: GND -> /SHIELD
- D1 pad 1: Net-(C4-Pad1) -> ROWA
- D1 pad 2: VBUS -> Net-(D1-Pad2)
- D10 pad 1: ROW0 -> ROWA
- D11 pad 1: ROW0 -> ROWA
- D12 pad 1: ROW0 -> ROWA
- D13 pad 1: ROW1 -> ROWB
- D14 pad 1: ROW1 -> ROWB
- D15 pad 1: ROW1 -> ROWB
- D16 pad 1: ROW1 -> ROWB
- D17 pad 1: ROW1 -> ROWB
- D18 pad 1: ROW1 -> ROWB
- D19 pad 1: ROW1 -> ROWB
- D2 pad 1: Net-(D2-Pad1) -> ROWA
- D20 pad 1: ROW1 -> ROWB
- D21 pad 1: ROW1 -> ROWB
- D22 pad 1: ROW1 -> ROWB
- D23 pad 1: ROW2 -> ROWB
- D24 pad 1: ROW2 -> ROWB
- D25 pad 1: ROW2 -> ROWC
- D26 pad 1: ROW2 -> ROWC
- D27 pad 1: ROW2 -> ROWC
- D28 pad 1: ROW2 -> ROWC
- D29 pad 1: ROW2 -> ROWC
- D3 pad 1: ROW0 -> ROWA
- D30 pad 1: ROW2 -> ROWC
- D31 pad 1: ROW2 -> ROWC
- D32 pad 1: ROW2 -> ROWC
- D33 pad 1: ROW3 -> ROWC
- D34 pad 1: ROW3 -> ROWC
- D35 pad 1: ROW3 -> ROWC
- D36 pad 1: ROW3 -> ROWC
- D37 pad 1: ROW3 -> ROWD
- D38 pad 1: ROW3 -> ROWD
- D39 pad 1: Net-(D39-Pad1) -> ROWD
- D39 pad 2: LED_1 -> Net-(D39-Pad2)
- D4 pad 1: ROW0 -> ROWA
- D40 pad 1: GND -> ROWD
- D40 pad 2: D- -> Net-(D40-Pad2)
- D5 pad 1: ROW0 -> ROWA
- D6 pad 1: ROW0 -> ROWA
- D7 pad 1: ROW0 -> ROWA
- D8 pad 1: ROW0 -> ROWA
- D9 pad 1: ROW0 -> ROWA
- F1 pad 2: RAW -> /RAW
- H1 pad 1: Net-(H1-Pad1) -> (no net)
- H2 pad 1: Net-(H2-Pad1) -> (no net)
- H3 pad 1: Net-(H3-Pad1) -> (no net)
- H4 pad 1: Net-(H4-Pad1) -> (no net)
- H5 pad 1: Net-(H5-Pad1) -> (no net)
- H6 pad 1: Net-(H6-Pad1) -> (no net)
- H7 pad 1: Net-(H7-Pad1) -> (no net)
- H8 pad 1: Net-(H8-Pad1) -> (no net)
- Q1 pad 2: Net-(C4-Pad1) -> /PVIN
- R3 pad 1: GND -> Net-(R3-Pad1)
- R3 pad 2: Net-(R3-Pad2) -> GND
- R4 pad 1: VBUS -> Net-(R4-Pad1)
- R4 pad 2: Net-(D2-Pad2) -> GND
- R5 pad 1: GND -> Net-(D45-Pad1)
- R5 pad 2: Net-(R5-Pad2) -> /charge
- R6 pad 2: Earth -> /SHIELD
- R7 pad 1: BVOLT -> Net-(D46-Pad1)
- R7 pad 2: VBAT -> GND
- R8 pad 1: GND -> VTAP
- R8 pad 2: BVOLT -> VBAT
- R9 pad 1: Net-(D39-Pad1) -> GND
- R9 pad 2: GND -> VTAP
- U2 pad 1: Net-(C4-Pad1) -> /PVIN
- U2 pad 3: Net-(C4-Pad1) -> /PVIN
- U2 pad 4: Net-(U2-Pad4) -> unconnected-(U2-Pad4)
- U3 pad 1: Net-(D2-Pad1) -> GND
- U3 pad 2: GND -> enc2B
- U3 pad 3: VBAT -> enc2A
- U3 pad 4: VBUS -> COL11
- U3 pad 5: Net-(R3-Pad2) -> COL10
Routing:
- net ROW1: track 356.6 -> 0.00 mm, vias 12 -> 0
- net ROW0: track 354.1 -> 0.00 mm, vias 12 -> 0
- net ROW2: track 326.7 -> 0.00 mm, vias 13 -> 0
- net ROWA: track 0.00 -> 321.6 mm, vias 0 -> 15
- net ROWC: track 0.00 -> 304.9 mm, vias 0 -> 15
- net ROWB: track 0.00 -> 293.0 mm, vias 0 -> 14
- net ROW3: track 195.5 -> 0.00 mm, vias 8 -> 0
- net ROWD: track 0.00 -> 193.6 mm, vias 0 -> 8
- net COL00: track 0.00 -> 162.6 mm, vias 0 -> 2
- net COL0: track 162.5 -> 0.00 mm, vias 1 -> 0
- net COL11: track 0.00 -> 153.5 mm, vias 0 -> 1
- net COL03: track 0.00 -> 152.7 mm, vias 0 -> 2
- net COL9: track 152.2 -> 0.00 mm, vias 1 -> 0
- net COL1: track 147.4 -> 0.00 mm, vias 1 -> 0
- net COL01: track 0.00 -> 143.9 mm, vias 0 -> 2
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Other:
- board size 265.7 x 104.1 mm -> 252.3 x 111.8 mm
- net class Default removed
- net class Power removed
- board text added: "+V"
- board text removed: "+"
- board text removed: "-"
- board text removed: "VBUS"
