File: revlp/one42/one42_pcb/one42.kicad_pcb (KiCad board)
At the start: 2 copper layers, 252.3 x 111.8 mm, 121 parts, among them J1 Conn_01x04_Female, Q1 AO3401A, SW44 SW_SPDT, U1 TP4054, U2 AP2112K-3.3, U3 nRF52840_holyiot_18010, U4 One42

Commit message: [keyboard] One42: Version 1.0
Parts:
- removed H1, H2, H3, H4, H5, H6, H7, H8: MountingHole, MountingHole:MountingHole_2.2mm_M2_Pad
- removed JP1: EncoderPolarity, Jumper:SolderJumper-3_P1.3mm_Open_RoundedPad1.0x1.5mm
- moved U1 16.2 mm to (72.4, 107.1), turned to -165 degrees
- moved R2 15.8 mm to (44.1, 67.7), turned to 0 degrees
- moved R4 14.9 mm to (68.0, 109.1), turned to -165 degrees
- moved BT1 12.9 mm to (61.5, 112.2), turned to 180 degrees
- moved SwC11 12.3 mm to (161.3, 77.3)
- moved SwC05 12.3 mm to (23.7, 96.8)
- moved R5 12.3 mm to (56.9, 49.0)
- moved SW44 12.3 mm to (72.5, 39.5)
- moved D45 12.3 mm to (53.5, 42.3)
- moved SwD04 12.3 mm to (17.2, 115.5)
- moved D12 12.3 mm to (150.3, 36.2)
- moved D1 12.3 mm to (-57.3, 36.2)
- moved D17 12.3 mm to (13.0, 64.1)
- moved F1 12.3 mm to (53.9, 49.5)
- moved D36 12.3 mm to (160.0, 72.5)
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Connections:
- net /PVIN renamed /VSRC
- net Net-(BT1-Pad2) renamed /BattSw
- J1 pad 1: VBUS -> VDD_NRF
- SwD03 pad C: /encBASE -> GND
- SwD08 pad C: /encBASE -> GND
Routing:
- net /encBASE: track 113.5 -> 0.00 mm, vias 1 -> 0
- net VBUS: track 129.9 -> 90.9 mm, vias 3 -> 2
- net VDD_NRF: track 11.9 -> 47.6 mm, vias 0 -> 2
- net /charge: track 59.6 -> 66.0 mm
- net VBAT: track 82.4 -> 86.8 mm
- net SWC: track 30.0 -> 25.7 mm, vias 1 -> 0
- net COL06: track 90.1 -> 86.1 mm
- net SWD: track 31.1 -> 27.4 mm, vias 1 -> 0
- net /BattSw: track 93.1 -> 95.2 mm
- net Net-(R4-Pad1): track 4.79 -> 2.77 mm
- net ROWC: track 304.9 -> 302.9 mm
- net ROWA: track 321.6 -> 320.0 mm
- net ROWB: track 293.0 -> 291.5 mm
- net /VSRC: track 11.9 -> 13.3 mm
- net RESET: track 46.8 -> 45.9 mm
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Other:
- board text added: "+3v3"
